Commit message: Modify the collision of barista to correct form

File: universal_robot_ros2/barista_ros2/barista_description/robot/barista_mod.xacro (robot description, xacro)
@@ -24,5 +24,5 @@
         <origin xyz="0 0 0" rpy="0 0 0"/>
         <geometry>
-          <mesh filename="package://barista_description/meshes/barista/TOP_collision_lip_sd.stl"/>
+          <mesh filename="package://barista_description/meshes/barista/TOP_colour_1.dae"/>
         </geometry>
       </collision>
