Commit message: Add the second camera for coffee position

File: universal_robot_ros2/Universal_Robots_ROS2_Description/urdf/ur.urdf.xacro (robot description, xacro)
@@ -97,4 +97,7 @@
        <origin xyz="-0.2 -0.3 0.2" rpy="0 ${pi/3} ${pi/2}"/>
    </xacro:sensor_r430>
+    <xacro:sensor_r430 prefix="camera" parent="base_link" >
+       <origin xyz="0.8 0.5 0.2" rpy="0 ${pi/6} ${pi}"/>
+   </xacro:sensor_r430>
    <xacro:if value="$(arg sim_gazebo)">
     <!-- Gazebo plugins -->

Commit message: Simulate the cup position in real lab succeed to grasp four cups to robots

File: universal_robot_ros2/Universal_Robots_ROS2_Description/urdf/ur.urdf.xacro (robot description, xacro)
@@ -95,5 +95,6 @@
    </xacro:rg2_gripper>
    <xacro:sensor_r430 prefix="wrist_rgbd" parent="base_link" >
-       <origin xyz="-0.2 -0.3 0.2" rpy="0 ${pi/3} ${pi/2}"/>
+       <!-- <origin xyz="-0.2 -0.3 0.2" rpy="0 ${pi/3} ${pi/2}"/> -->
+       <origin xyz="-0.25 -0.3 0.2" rpy="0 ${pi/3} ${pi/2}"/>
    </xacro:sensor_r430>
     <xacro:sensor_r430 prefix="camera" parent="base_link" >
